File: boards/gp4-hil/gp4-hil.sch (KiCad schematic (older format))
At the start: 23 parts

Commit message: Began work on footprint creation for layout.
Parts:
- JP1, JP2, JP3, JP4, JP5, JP6: footprint (none) -> azonenberg_pcb:JUMPER_2.54MM_2POS
- TP34, TP35, TP36: footprint (none) -> azonenberg_pcb:TESTPOINT_SMT_KEYSTONE_5016
Changed lines of the file:
@@
 F 0 "R170" V 3700 3350 50  0000 C CNN
 F 1 "10K" V 3750 3150 50  0000 C CNN
-F 2 "" V 3680 3150 30  0000 C CNN
+F 2 "" V 3680 3150 30  0001 C CNN
 F 3 "" H 3750 3150 30  0000 C CNN
 	1    3750 3150
@@
 F 0 "R171" V 3700 3450 50  0000 C CNN
 F 1 "10K" V 3750 3250 50  0000 C CNN
-F 2 "" V 3680 3250 30  0000 C CNN
+F 2 "" V 3680 3250 30  0001 C CNN
 F 3 "" H 3750 3250 30  0000 C CNN
 	1    3750 3250
@@
 F 0 "R172" V 3700 3550 50  0000 C CNN
 F 1 "10K" V 3750 3350 50  0000 C CNN
-F 2 "" V 3680 3350 30  0000 C CNN
+F 2 "" V 3680 3350 30  0001 C CNN
 F 3 "" H 3750 3350 30  0000 C CNN
 	1    3750 3350
@@
 F 0 "R173" V 3700 3750 50  0000 C CNN
 F 1 "10K" V 3750 3550 50  0000 C CNN
-F 2 "" V 3680 3550 30  0000 C CNN
+F 2 "" V 3680 3550 30  0001 C CNN
 F 3 "" H 3750 3550 30  0000 C CNN
 	1    3750 3550
@@
 F 0 "R174" V 3700 3850 50  0000 C CNN
 F 1 "10K" V 3750 3650 50  0000 C CNN
-F 2 "" V 3680 3650 30  0000 C CNN
+F 2 "" V 3680 3650 30  0001 C CNN
 F 3 "" H 3750 3650 30  0000 C CNN
 	1    3750 3650
@@
 F 0 "R175" V 3700 3950 50  0000 C CNN
 F 1 "10K" V 3750 3750 50  0000 C CNN
-F 2 "" V 3680 3750 30  0000 C CNN
+F 2 "" V 3680 3750 30  0001 C CNN
 F 3 "" H 3750 3750 30  0000 C CNN
 	1    3750 3750
@@
 F 0 "R176" V 3700 4150 50  0000 C CNN
 F 1 "1K" V 3750 3950 50  0000 C CNN
-F 2 "" V 3680 3950 30  0000 C CNN
+F 2 "" V 3680 3950 30  0001 C CNN
 F 3 "" H 3750 3950 30  0000 C CNN
 	1    3750 3950
@@
 F 0 "R169" V 3650 6950 50  0000 C CNN
 F 1 "1K" V 3700 6750 50  0000 C CNN
-F 2 "" V 3630 6750 30  0000 C CNN
+F 2 "" V 3630 6750 30  0001 C CNN
 F 3 "" H 3700 6750 30  0000 C CNN
 	1    3700 6750
@@
 F 0 "JP1" H 7250 7550 50  0000 C CNN
 F 1 "JUMPER" H 7700 7550 50  0000 C CNN
-F 2 "" H 7450 7400 60  0000 C CNN
+F 2 "azonenberg_pcb:JUMPER_2.54MM_2POS" H 7450 7400 60  0001 C CNN
 F 3 "" H 7450 7400 60  0000 C CNN
 	1    7450 7400
@@
 F 0 "JP2" H 7250 7800 50  0000 C CNN
 F 1 "JUMPER" H 7700 7800 50  0000 C CNN
-F 2 "" H 7450 7650 60  0000 C CNN
+F 2 "azonenberg_pcb:JUMPER_2.54MM_2POS" H 7450 7650 60  0001 C CNN
 F 3 "" H 7450 7650 60  0000 C CNN
 	1    7450 7650
@@
 F 0 "JP3" H 7250 8050 50  0000 C CNN
 F 1 "JUMPER" H 7700 8050 50  0000 C CNN
-F 2 "" H 7450 7900 60  0000 C CNN
+F 2 "azonenberg_pcb:JUMPER_2.54MM_2POS" H 7450 7900 60  0001 C CNN
 F 3 "" H 7450 7900 60  0000 C CNN
 	1    7450 7900
@@
 F 0 "JP4" H 7250 8300 50  0000 C CNN
 F 1 "JUMPER" H 7700 8300 50  0000 C CNN
-F 2 "" H 7450 8150 60  0000 C CNN
+F 2 "azonenberg_pcb:JUMPER_2.54MM_2POS" H 7450 8150 60  0001 C CNN
 F 3 "" H 7450 8150 60  0000 C CNN
 	1    7450 8150
@@
 F 0 "JP5" H 7250 8550 50  0000 C CNN
 F 1 "JUMPER" H 7700 8550 50  0000 C CNN
-F 2 "" H 7450 8400 60  0000 C CNN
+F 2 "azonenberg_pcb:JUMPER_2.54MM_2POS" H 7450 8400 60  0001 C CNN
 F 3 "" H 7450 8400 60  0000 C CNN
 	1    7450 8400
@@
 F 0 "JP6" H 7250 8800 50  0000 C CNN
 F 1 "JUMPER" H 7700 8800 50  0000 C CNN
-F 2 "" H 7450 8650 60  0000 C CNN
+F 2 "azonenberg_pcb:JUMPER_2.54MM_2POS" H 7450 8650 60  0001 C CNN
 F 3 "" H 7450 8650 60  0000 C CNN
 	1    7450 8650
@@
 F 0 "R181" V 7900 7550 50  0000 C CNN
 F 1 "1K" V 8000 7400 50  0000 C CNN
-F 2 "" V 7930 7400 30  0000 C CNN
+F 2 "" V 7930 7400 30  0001 C CNN
 F 3 "" H 8000 7400 30  0000 C CNN
 	1    8000 7400
@@
 F 0 "R182" V 7900 7800 50  0000 C CNN
 F 1 "1K" V 8000 7650 50  0000 C CNN
-F 2 "" V 7930 7650 30  0000 C CNN
+F 2 "" V 7930 7650 30  0001 C CNN
 F 3 "" H 8000 7650 30  0000 C CNN
 	1    8000 7650
@@
 F 0 "R183" V 7900 8050 50  0000 C CNN
 F 1 "1K" V 8000 7900 50  0000 C CNN
-F 2 "" V 7930 7900 30  0000 C CNN
+F 2 "" V 7930 7900 30  0001 C CNN
 F 3 "" H 8000 7900 30  0000 C CNN
 	1    8000 7900
@@
 F 0 "R184" V 7900 8300 50  0000 C CNN
 F 1 "1K" V 8000 8150 50  0000 C CNN
-F 2 "" V 7930 8150 30  0000 C CNN
+F 2 "" V 7930 8150 30  0001 C CNN
 F 3 "" H 8000 8150 30  0000 C CNN
 	1    8000 8150
@@
 F 0 "R185" V 7900 8550 50  0000 C CNN
 F 1 "1K" V 8000 8400 50  0000 C CNN
-F 2 "" V 7930 8400 30  0000 C CNN
+F 2 "" V 7930 8400 30  0001 C CNN
 F 3 "" H 8000 8400 30  0000 C CNN
 	1    8000 8400
@@
 F 0 "R186" V 7900 8800 50  0000 C CNN
 F 1 "1K" V 8000 8650 50  0000 C CNN
-F 2 "" V 7930 8650 30  0000 C CNN
+F 2 "" V 7930 8650 30  0001 C CNN
 F 3 "" H 8000 8650 30  0000 C CNN
 	1    8000 8650
@@
 F 0 "TP36" H 10100 8650 50  0000 C CNN
 F 1 "TESTPOINT" H 9600 8600 50  0000 C CNN
-F 2 "" H 9950 8650 60  0000 C CNN
+F 2 "azonenberg_pcb:TESTPOINT_SMT_KEYSTONE_5016" H 9950 8650 60  0001 C CNN
 F 3 "" H 9950 8650 60  0000 C CNN
 	1    9950 8650
@@
 F 0 "TP35" H 10100 8400 50  0000 C CNN
 F 1 "TESTPOINT" H 9600 8350 50  0000 C CNN
-F 2 "" H 9950 8400 60  0000 C CNN
+F 2 "azonenberg_pcb:TESTPOINT_SMT_KEYSTONE_5016" H 9950 8400 60  0001 C CNN
 F 3 "" H 9950 8400 60  0000 C CNN
 	1    9950 8400
@@
 F 0 "TP34" H 10100 8150 50  0000 C CNN
 F 1 "TESTPOINT" H 9600 8100 50  0000 C CNN
-F 2 "" H 9950 8150 60  0000 C CNN
+F 2 "azonenberg_pcb:TESTPOINT_SMT_KEYSTONE_5016" H 9950 8150 60  0001 C CNN
 F 3 "" H 9950 8150 60  0000 C CNN
 	1    9950 8150
