File: boards/gp4-hil/psu.sch (KiCad schematic (older format))
At the start: 81 parts, among them K1 CONN_3_PWROUT, Q11 SSM6N58NU, Q12 DMP2069UFY4, Q22 DMP2069UFY4, U1 MIC2288-DFN, U20 SIP32408, U21 SIP32408, U22 SIP32408, U23 SIP32408, U24 SIP32408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

Commit message: Began work on footprint creation for layout.
Parts:
- C116, C117, C118, C119, C120, C121, C123, C124, C125, C126, C127, C128, C129, C130: footprint (none) -> azonenberg_pcb:EIA_1206_CAP_NOSILK
- C122, L12: footprint (none) -> azonenberg_pcb:EIA_1210_CAP_NOSILK
- C131, C132, C133, C137, C138, C139, C171: footprint (none) -> azonenberg_pcb:EIA_0603_CAP_NOSILK
- C134, C135, C136, C140, C141, C142, C172: footprint (none) -> azonenberg_pcb:EIA_0402_CAP_NOSILK
- D20: footprint (none) -> azonenberg_pcb:EIA_0402_LED
- D39: footprint (none) -> azonenberg_pcb:EIA_0603_LED
- F1: footprint (none) -> azonenberg_pcb:EIA_0402_RES_NOSILK
- K1: footprint (none) -> azonenberg_pcb:CONN_CUI_PJ-058BH_HIPWR_BARREL_NOSLOT
- L10, L11, L7, L9: footprint (none) -> azonenberg_pcb:INDUCTOR_YUDEN_NR6028
- L6: footprint (none) -> azonenberg_pcb:INDUCTOR_TDK_SPM6530
- L8: footprint (none) -> azonenberg_pcb:EIA_0805_INDUCTOR_NOSILK
- Q11: footprint (none) -> azonenberg_pcb:DFN_6_0.65MM_2x2MM_GDS
- TP24, TP25, TP26, TP27, TP28, TP29, TP30, TP31, TP32: footprint (none) -> azonenberg_pcb:TESTPOINT_SMT_KEYSTONE_5016

Commit message: Updated PCB with a lot more component footprints
Parts:
- L8: footprint azonenberg_pcb:EIA_0805_INDUCTOR_NOSILK -> azonenberg_pcb:EIA_0603_INDUCTOR_NOSILK
- R100, R113, R114, R177: footprint (none) -> azonenberg_pcb:EIA_0402_RES_NOSILK
- U3: footprint (none) -> azonenberg_pcb:QFN_38_0.5MM_5x7MM
Changed lines of the file:
@@
 Sheet 2 7
 Title "GreenPak Hardware-In-Loop Test Platform"
-Date "2016-05-19"
+Date "2016-05-20"
 Rev "0.1"
 Comp "Andrew Zonenberg"
@@
 F 0 "U3" H 3750 5050 60  0000 L CNN
 F 1 "LTC3374-QFN" H 3000 5050 60  0000 L CNN
-F 2 "" H 3000 5100 60  0001 C CNN
+F 2 "azonenberg_pcb:QFN_38_0.5MM_5x7MM" H 3000 5100 60  0001 C CNN
 F 3 "" H 3000 5100 60  0000 C CNN
 	2    3000 5100
@@
 F 0 "U3" H 3750 4200 60  0000 L CNN
 F 1 "LTC3374-QFN" H 3000 4200 60  0000 L CNN
-F 2 "" H 3000 4250 60  0001 C CNN
+F 2 "azonenberg_pcb:QFN_38_0.5MM_5x7MM" H 3000 4250 60  0001 C CNN
 F 3 "" H 3000 4250 60  0000 C CNN
 	1    3000 4250
@@
 F 0 "U3" H 3750 5900 60  0000 L CNN
 F 1 "LTC3374-QFN" H 3000 5900 60  0000 L CNN
-F 2 "" H 3000 5950 60  0001 C CNN
+F 2 "azonenberg_pcb:QFN_38_0.5MM_5x7MM" H 3000 5950 60  0001 C CNN
 F 3 "" H 3000 5950 60  0000 C CNN
 	3    3000 5950
@@
 F 0 "U3" H 3750 6750 60  0000 L CNN
 F 1 "LTC3374-QFN" H 3000 6750 60  0000 L CNN
-F 2 "" H 3000 6800 60  0001 C CNN
+F 2 "azonenberg_pcb:QFN_38_0.5MM_5x7MM" H 3000 6800 60  0001 C CNN
 F 3 "" H 3000 6800 60  0000 C CNN
 	4    3000 6800
@@
 F 0 "U3" H 3750 7700 60  0000 L CNN
 F 1 "LTC3374-QFN" H 3000 7700 60  0000 L CNN
-F 2 "" H 3000 7750 60  0001 C CNN
+F 2 "azonenberg_pcb:QFN_38_0.5MM_5x7MM" H 3000 7750 60  0001 C CNN
 F 3 "" H 3000 7750 60  0000 C CNN
 	5    3000 7750
@@
 F 0 "U3" H 3750 8650 60  0000 L CNN
 F 1 "LTC3374-QFN" H 3000 8650 60  0000 L CNN
-F 2 "" H 3000 8700 60  0001 C CNN
+F 2 "azonenberg_pcb:QFN_38_0.5MM_5x7MM" H 3000 8700 60  0001 C CNN
 F 3 "" H 3000 8700 60  0000 C CNN
 	6    3000 8700
@@
 F 0 "U3" H 2550 2803 60  0000 C CNN
 F 1 "LTC3374-QFN" H 2550 2697 60  0000 C CNN
-F 2 "" H 2100 2100 60  0001 C CNN
+F 2 "azonenberg_pcb:QFN_38_0.5MM_5x7MM" H 2100 2100 60  0001 C CNN
 F 3 "" H 2100 2100 60  0000 C CNN
 	9    2100 2100
@@
 F 0 "R100" V 3950 1600 50  0000 C CNN
 F 1 "1K" V 4050 1600 50  0000 C CNN
-F 2 "" V 3980 1600 30  0001 C CNN
+F 2 "azonenberg_pcb:EIA_0402_RES_NOSILK" V 3980 1600 30  0001 C CNN
 F 3 "" H 4050 1600 30  0000 C CNN
 	1    4050 1600
@@
 F 0 "L8" V 3850 15350 40  0000 C CNN
 F 1 "600R" V 3850 14900 40  0000 C CNN
-F 2 "azonenberg_pcb:EIA_0805_INDUCTOR_NOSILK" H 3900 15100 60  0001 C CNN
+F 2 "azonenberg_pcb:EIA_0603_INDUCTOR_NOSILK" H 3900 15100 60  0001 C CNN
 F 3 "" H 3900 15100 60  0000 C CNN
 	1    3900 15100
@@
 F 0 "U3" H 3750 9600 60  0000 L CNN
 F 1 "LTC3374-QFN" H 3000 9600 60  0000 L CNN
-F 2 "" H 3000 9650 60  0001 C CNN
+F 2 "azonenberg_pcb:QFN_38_0.5MM_5x7MM" H 3000 9650 60  0001 C CNN
 F 3 "" H 3000 9650 60  0000 C CNN
 	7    3000 9650
@@
 F 0 "U3" H 3750 10550 60  0000 L CNN
 F 1 "LTC3374-QFN" H 3000 10550 60  0000 L CNN
-F 2 "" H 3000 10600 60  0001 C CNN
+F 2 "azonenberg_pcb:QFN_38_0.5MM_5x7MM" H 3000 10600 60  0001 C CNN
 F 3 "" H 3000 10600 60  0000 C CNN
 	8    3000 10600
@@
 F 0 "R113" H 9270 4646 50  0000 L CNN
 F 1 "4.7K 1%" H 9270 4554 50  0000 L CNN
-F 2 "" V 9130 4600 30  0001 C CNN
+F 2 "azonenberg_pcb:EIA_0402_RES_NOSILK" V 9130 4600 30  0001 C CNN
 F 3 "" H 9200 4600 30  0000 C CNN
 	1    9200 4600
@@
 F 0 "R114" H 11520 4196 50  0000 L CNN
 F 1 "1K" H 11520 4104 50  0000 L CNN
-F 2 "" V 11380 4150 30  0001 C CNN
+F 2 "azonenberg_pcb:EIA_0402_RES_NOSILK" V 11380 4150 30  0001 C CNN
 F 3 "" H 11450 4150 30  0000 C CNN
 	1    11450 4150
@@
 F 0 "R177" H 4470 15396 50  0000 L CNN
 F 1 "470" H 4470 15304 50  0000 L CNN
-F 2 "" V 4330 15350 30  0001 C CNN
+F 2 "azonenberg_pcb:EIA_0402_RES_NOSILK" V 4330 15350 30  0001 C CNN
 F 3 "" H 4400 15350 30  0000 C CNN
 	1    4400 15350

Commit message: More footprint assignments
Parts:
- Q12, Q22: footprint (none) -> azonenberg_pcb:DFN_3_DIODES_X2DFN2015-3
- R101, R102, R103, R104, R105, R106, R107, R108, R109, R110, R111, R112, R115, R116, R117, R118, R179: footprint (none) -> azonenberg_pcb:EIA_0402_RES_NOSILK
Changed lines of the file:
@@
 F 0 "R101" V 4050 4950 50  0000 C CNN
 F 1 "2.55K" V 4000 4750 50  0000 C CNN
-F 2 "" V 4030 4750 30  0001 C CNN
+F 2 "azonenberg_pcb:EIA_0402_RES_NOSILK" V 4030 4750 30  0001 C CNN
 F 3 "" H 4100 4750 30  0000 C CNN
 	1    4100 4750
@@
 F 0 "R102" V 4050 5100 50  0000 C CNN
 F 1 "10.2K" V 4200 4900 50  0000 C CNN
-F 2 "" V 4030 4900 30  0001 C CNN
+F 2 "azonenberg_pcb:EIA_0402_RES_NOSILK" V 4030 4900 30  0001 C CNN
 F 3 "" H 4100 4900 30  0000 C CNN
 	1    4100 4900
@@
 F 0 "R103" V 4800 4950 50  0000 C CNN
 F 1 "0" V 4850 4750 50  0000 C CNN
-F 2 "" V 4780 4750 30  0001 C CNN
+F 2 "azonenberg_pcb:EIA_0402_RES_NOSILK" V 4780 4750 30  0001 C CNN
 F 3 "" H 4850 4750 30  0000 C CNN
 	1    4850 4750
@@
 F 0 "R104" V 3500 7500 50  0000 C CNN
 F 1 "232K" V 3550 7700 50  0000 C CNN
-F 2 "" V 3480 7700 30  0001 C CNN
+F 2 "azonenberg_pcb:EIA_0402_RES_NOSILK" V 3480 7700 30  0001 C CNN
 F 3 "" H 3550 7700 30  0000 C CNN
 	1    3550 7700
@@
 F 0 "R105" V 3500 8000 50  0000 C CNN
 F 1 "464K" V 3550 7800 50  0000 C CNN
-F 2 "" V 3480 7800 30  0001 C CNN
+F 2 "azonenberg_pcb:EIA_0402_RES_NOSILK" V 3480 7800 30  0001 C CNN
 F 3 "" H 3550 7800 30  0000 C CNN
 	1    3550 7800
@@
 F 0 "R106" V 3500 8450 50  0000 C CNN
 F 1 "806K" V 3550 8650 50  0000 C CNN
-F 2 "" V 3480 8650 30  0001 C CNN
+F 2 "azonenberg_pcb:EIA_0402_RES_NOSILK" V 3480 8650 30  0001 C CNN
 F 3 "" H 3550 8650 30  0000 C CNN
 	1    3550 8650
@@
 F 0 "R107" V 3500 8950 50  0000 C CNN
 F 1 "649K" V 3550 8750 50  0000 C CNN
-F 2 "" V 3480 8750 30  0001 C CNN
+F 2 "azonenberg_pcb:EIA_0402_RES_NOSILK" V 3480 8750 30  0001 C CNN
 F 3 "" H 3550 8750 30  0000 C CNN
 	1    3550 8750
@@
 F 0 "R108" V 3500 9400 50  0000 C CNN
 F 1 "1.02M" V 3550 9600 50  0000 C CNN
-F 2 "" V 3480 9600 30  0001 C CNN
+F 2 "azonenberg_pcb:EIA_0402_RES_NOSILK" V 3480 9600 30  0001 C CNN
 F 3 "" H 3550 9600 30  0000 C CNN
 	1    3550 9600
@@
 F 0 "R109" V 3500 9900 50  0000 C CNN
 F 1 "475K" V 3550 9700 50  0000 C CNN
-F 2 "" V 3480 9700 30  0001 C CNN
+F 2 "azonenberg_pcb:EIA_0402_RES_NOSILK" V 3480 9700 30  0001 C CNN
 F 3 "" H 3550 9700 30  0000 C CNN
 	1    3550 9700
@@
 F 0 "R110" V 3500 10350 50  0000 C CNN
 F 1 "1.02M" V 3550 10550 50  0000 C CNN
-F 2 "" V 3480 10550 30  0001 C CNN
+F 2 "azonenberg_pcb:EIA_0402_RES_NOSILK" V 3480 10550 30  0001 C CNN
 F 3 "" H 3550 10550 30  0000 C CNN
 	1    3550 10550
@@
 F 0 "R111" V 3500 10850 50  0000 C CNN
 F 1 "324K" V 3550 10650 50  0000 C CNN
-F 2 "" V 3480 10650 30  0001 C CNN
+F 2 "azonenberg_pcb:EIA_0402_RES_NOSILK" V 3480 10650 30  0001 C CNN
 F 3 "" H 3550 10650 30  0000 C CNN
 	1    3550 10650
@@
 F 0 "R112" H 9270 4196 50  0000 L CNN
 F 1 "24K 1%" H 9270 4104 50  0000 L CNN
-F 2 "" V 9130 4150 30  0001 C CNN
+F 2 "azonenberg_pcb:EIA_0402_RES_NOSILK" V 9130 4150 30  0001 C CNN
 F 3 "" H 9200 4150 30  0000 C CNN
 	1    9200 4150
@@
 F 0 "Q12" H 12444 4304 50  0000 L CNN
 F 1 "DMP2069UFY4" H 12444 4396 50  0000 L CNN
-F 2 "" H 12450 4450 29  0001 C CNN
+F 2 "azonenberg_pcb:DFN_3_DIODES_X2DFN2015-3" H 12450 4450 29  0001 C CNN
 F 3 "" H 12250 4350 60  0000 C CNN
 	1    12250 4350
@@
 F 0 "R116" H 9370 8696 50  0000 L CNN
 F 1 "0" H 9370 8604 50  0000 L CNN
-F 2 "" V 9230 8650 30  0001 C CNN
+F 2 "azonenberg_pcb:EIA_0402_RES_NOSILK" V 9230 8650 30  0001 C CNN
 F 3 "" H 9300 8650 30  0000 C CNN
 	1    9300 8650
@@
 F 0 "R115" H 9370 7946 50  0000 L CNN
 F 1 "0" H 9370 7854 50  0000 L CNN
-F 2 "" V 9230 7900 30  0001 C CNN
+F 2 "azonenberg_pcb:EIA_0402_RES_NOSILK" V 9230 7900 30  0001 C CNN
 F 3 "" H 9300 7900 30  0000 C CNN
 	1    9300 7900
@@
 F 0 "R117" H 14470 7946 50  0000 L CNN
 F 1 "0" H 14470 7854 50  0000 L CNN
-F 2 "" V 14330 7900 30  0001 C CNN
+F 2 "azonenberg_pcb:EIA_0402_RES_NOSILK" V 14330 7900 30  0001 C CNN
 F 3 "" H 14400 7900 30  0000 C CNN
 	1    14400 7900
@@
 F 0 "R118" H 14470 8696 50  0000 L CNN
 F 1 "0" H 14470 8604 50  0000 L CNN
-F 2 "" V 14330 8650 30  0001 C CNN
+F 2 "azonenberg_pcb:EIA_0402_RES_NOSILK" V 14330 8650 30  0001 C CNN
 F 3 "" H 14400 8650 30  0000 C CNN
 	1    14400 8650
@@
 F 0 "Q22" V 3200 15000 50  0000 C CNN
 F 1 "DMP2069UFY4" V 3100 14800 50  0000 C CNN
-F 2 "" H 3400 15300 29  0001 C CNN
+F 2 "azonenberg_pcb:DFN_3_DIODES_X2DFN2015-3" H 3400 15300 29  0001 C CNN
 F 3 "" H 3200 15200 60  0000 C CNN
 	1    3200 15200
@@
 F 0 "R179" V 13650 4750 50  0000 C CNN
 F 1 "0.1" V 13700 4550 50  0000 C CNN
-F 2 "" V 13630 4550 30  0001 C CNN
+F 2 "azonenberg_pcb:EIA_0402_RES_NOSILK" V 13630 4550 30  0001 C CNN
 F 3 "" H 13700 4550 30  0000 C CNN
 	1    13700 4550

Commit message: Finished component footprints. Ready to begin layout.
Parts:
- U1: footprint (none) -> azonenberg_pcb:DFN_8_0.5MM_2x2MM
- U20, U21, U22, U23, U24, U4: footprint (none) -> azonenberg_pcb:DFN_4_0.5MM_1.6x1.2MM
Changed lines of the file:
@@
 Sheet 2 7
 Title "GreenPak Hardware-In-Loop Test Platform"
-Date "2016-05-20"
+Date "2016-05-22"
 Rev "0.1"
 Comp "Andrew Zonenberg"
@@
 F 0 "U1" H 7900 4750 60  0000 C CNN
 F 1 "MIC2288-DFN" H 8450 4750 60  0000 C CNN
-F 2 "" H 7850 4800 60  0001 C CNN
+F 2 "azonenberg_pcb:DFN_8_0.5MM_2x2MM" H 7850 4800 60  0001 C CNN
 F 3 "" H 7850 4800 60  0000 C CNN
 	1    7850 4800
@@
 F 0 "U4" H 7750 8050 60  0000 C CNN
 F 1 "SIP32408" H 8100 8050 60  0000 C CNN
-F 2 "" H 7700 8100 60  0001 C CNN
+F 2 "azonenberg_pcb:DFN_4_0.5MM_1.6x1.2MM" H 7700 8100 60  0001 C CNN
 F 3 "" H 7700 8100 60  0000 C CNN
 	1    7700 8100
@@
 F 0 "U21" H 7750 9550 60  0000 C CNN
 F 1 "SIP32408" H 8100 9550 60  0000 C CNN
-F 2 "" H 7700 9600 60  0001 C CNN
+F 2 "azonenberg_pcb:DFN_4_0.5MM_1.6x1.2MM" H 7700 9600 60  0001 C CNN
 F 3 "" H 7700 9600 60  0000 C CNN
 	1    7700 9600
@@
 F 0 "U20" H 7750 8800 60  0000 C CNN
 F 1 "SIP32408" H 8100 8800 60  0000 C CNN
-F 2 "" H 7700 8850 60  0001 C CNN
+F 2 "azonenberg_pcb:DFN_4_0.5MM_1.6x1.2MM" H 7700 8850 60  0001 C CNN
 F 3 "" H 7700 8850 60  0000 C CNN
 	1    7700 8850
@@
 F 0 "U22" H 12850 8050 60  0000 C CNN
 F 1 "SIP32408" H 13200 8050 60  0000 C CNN
-F 2 "" H 12800 8100 60  0001 C CNN
+F 2 "azonenberg_pcb:DFN_4_0.5MM_1.6x1.2MM" H 12800 8100 60  0001 C CNN
 F 3 "" H 12800 8100 60  0000 C CNN
 	1    12800 8100
@@
 F 0 "U24" H 12850 9550 60  0000 C CNN
 F 1 "SIP32408" H 13200 9550 60  0000 C CNN
-F 2 "" H 12800 9600 60  0001 C CNN
+F 2 "azonenberg_pcb:DFN_4_0.5MM_1.6x1.2MM" H 12800 9600 60  0001 C CNN
 F 3 "" H 12800 9600 60  0000 C CNN
 	1    12800 9600
@@
 F 0 "U23" H 12850 8800 60  0000 C CNN
 F 1 "SIP32408" H 13200 8800 60  0000 C CNN
-F 2 "" H 12800 8850 60  0001 C CNN
+F 2 "azonenberg_pcb:DFN_4_0.5MM_1.6x1.2MM" H 12800 8850 60  0001 C CNN
 F 3 "" H 12800 8850 60  0000 C CNN
 	1    12800 8850
