File: boards/gp4-hil/dut.sch (KiCad schematic (older format))
At the start: 77 parts, among them P1 GPAK_ZIF, P2 2x10 HEADER, Q11 SSM6N58NU, Q13 SSM6N58NU, Q14 SSM6N58NU, Q15 SSM6N58NU, Q16 SSM6N58NU, Q17 SSM6N58NU, Q18 SSM6N58NU, Q19 SSM6N58NU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

Commit message: Began work on footprint creation for layout.
Parts:
- C173: footprint (none) -> azonenberg_pcb:EIA_0603_CAP_NOSILK
- C174, C182, C183: footprint (none) -> azonenberg_pcb:EIA_0402_CAP_NOSILK
- D21, D22, D23, D24, D25, D26, D27, D28, D29, D30, D31, D32, D33, D34, D35, D36, D37, D38: footprint (none) -> azonenberg_pcb:EIA_0603_LED
- P1, P2: footprint (none) -> azonenberg_pcb:CONN_HEADER_2.54MM_2x10_RA_BRORIG
- Q11, Q13, Q14, Q15, Q16, Q17, Q18, Q19, Q20, Q21: footprint (none) -> azonenberg_pcb:DFN_6_0.65MM_2x2MM_GDS
- TP1, TP10, TP11, TP12, TP13, TP14, TP15, TP16, TP17, TP18, TP19, TP2, TP20, TP21, TP3, TP33, TP4, TP5, TP6, TP7, TP8, TP9: footprint (none) -> azonenberg_pcb:TESTPOINT_SMT_KEYSTONE_5016

Commit message: Updated PCB with a lot more component footprints
Parts:
- R151, R152, R153, R154, R155, R156, R157, R158, R159, R160, R161, R162, R163, R164, R165, R166, R167, R168: footprint (none) -> azonenberg_pcb:EIA_0402_RES_NOSILK
Changed lines of the file:
@@
 Sheet 4 7
 Title "GreenPak Hardware-In-Loop Test Platform"
-Date "2016-05-19"
+Date "2016-05-20"
 Rev "0.1"
 Comp "Andrew Zonenberg"
@@
 F 0 "R151" H 5530 5704 50  0000 R CNN
 F 1 "220" H 5530 5796 50  0000 R CNN
-F 2 "" V 5530 5750 30  0001 C CNN
+F 2 "azonenberg_pcb:EIA_0402_RES_NOSILK" V 5530 5750 30  0001 C CNN
 F 3 "" H 5600 5750 30  0000 C CNN
 	1    5600 5750
@@
 F 0 "R153" H 6480 5704 50  0000 R CNN
 F 1 "220" H 6480 5796 50  0000 R CNN
-F 2 "" V 6480 5750 30  0001 C CNN
+F 2 "azonenberg_pcb:EIA_0402_RES_NOSILK" V 6480 5750 30  0001 C CNN
 F 3 "" H 6550 5750 30  0000 C CNN
 	1    6550 5750
@@
 F 0 "R155" H 7430 5704 50  0000 R CNN
 F 1 "220" H 7430 5796 50  0000 R CNN
-F 2 "" V 7430 5750 30  0001 C CNN
+F 2 "azonenberg_pcb:EIA_0402_RES_NOSILK" V 7430 5750 30  0001 C CNN
 F 3 "" H 7500 5750 30  0000 C CNN
 	1    7500 5750
@@
 F 0 "R157" H 8380 5704 50  0000 R CNN
 F 1 "220" H 8380 5796 50  0000 R CNN
-F 2 "" V 8380 5750 30  0001 C CNN
+F 2 "azonenberg_pcb:EIA_0402_RES_NOSILK" V 8380 5750 30  0001 C CNN
 F 3 "" H 8450 5750 30  0000 C CNN
 	1    8450 5750
@@
 F 0 "R159" H 9330 5704 50  0000 R CNN
 F 1 "220" H 9330 5796 50  0000 R CNN
-F 2 "" V 9330 5750 30  0001 C CNN
+F 2 "azonenberg_pcb:EIA_0402_RES_NOSILK" V 9330 5750 30  0001 C CNN
 F 3 "" H 9400 5750 30  0000 C CNN
 	1    9400 5750
@@
 F 0 "R161" H 10280 5704 50  0000 R CNN
 F 1 "220" H 10280 5796 50  0000 R CNN
-F 2 "" V 10280 5750 30  0001 C CNN
+F 2 "azonenberg_pcb:EIA_0402_RES_NOSILK" V 10280 5750 30  0001 C CNN
 F 3 "" H 10350 5750 30  0000 C CNN
 	1    10350 5750
@@
 F 0 "R163" H 11230 5704 50  0000 R CNN
 F 1 "220" H 11230 5796 50  0000 R CNN
-F 2 "" V 11230 5750 30  0001 C CNN
+F 2 "azonenberg_pcb:EIA_0402_RES_NOSILK" V 11230 5750 30  0001 C CNN
 F 3 "" H 11300 5750 30  0000 C CNN
 	1    11300 5750
@@
 F 0 "R165" H 12180 5704 50  0000 R CNN
 F 1 "220" H 12180 5796 50  0000 R CNN
-F 2 "" V 12180 5750 30  0001 C CNN
+F 2 "azonenberg_pcb:EIA_0402_RES_NOSILK" V 12180 5750 30  0001 C CNN
 F 3 "" H 12250 5750 30  0000 C CNN
 	1    12250 5750
@@
 F 0 "R167" H 13130 5704 50  0000 R CNN
 F 1 "220" H 13130 5796 50  0000 R CNN
-F 2 "" V 13130 5750 30  0001 C CNN
+F 2 "azonenberg_pcb:EIA_0402_RES_NOSILK" V 13130 5750 30  0001 C CNN
 F 3 "" H 13200 5750 30  0000 C CNN
 	1    13200 5750
@@
 F 0 "R152" H 5530 7404 50  0000 R CNN
 F 1 "220" H 5530 7496 50  0000 R CNN
-F 2 "" V 5530 7450 30  0001 C CNN
+F 2 "azonenberg_pcb:EIA_0402_RES_NOSILK" V 5530 7450 30  0001 C CNN
 F 3 "" H 5600 7450 30  0000 C CNN
 	1    5600 7450
@@
 F 0 "R154" H 6480 7404 50  0000 R CNN
 F 1 "220" H 6480 7496 50  0000 R CNN
-F 2 "" V 6480 7450 30  0001 C CNN
+F 2 "azonenberg_pcb:EIA_0402_RES_NOSILK" V 6480 7450 30  0001 C CNN
 F 3 "" H 6550 7450 30  0000 C CNN
 	1    6550 7450
@@
 F 0 "R156" H 7430 7404 50  0000 R CNN
 F 1 "220" H 7430 7496 50  0000 R CNN
-F 2 "" V 7430 7450 30  0001 C CNN
+F 2 "azonenberg_pcb:EIA_0402_RES_NOSILK" V 7430 7450 30  0001 C CNN
 F 3 "" H 7500 7450 30  0000 C CNN
 	1    7500 7450
@@
 F 0 "R158" H 8380 7404 50  0000 R CNN
 F 1 "220" H 8380 7496 50  0000 R CNN
-F 2 "" V 8380 7450 30  0001 C CNN
+F 2 "azonenberg_pcb:EIA_0402_RES_NOSILK" V 8380 7450 30  0001 C CNN
 F 3 "" H 8450 7450 30  0000 C CNN
 	1    8450 7450
@@
 F 0 "R160" H 9330 7404 50  0000 R CNN
 F 1 "220" H 9330 7496 50  0000 R CNN
-F 2 "" V 9330 7450 30  0001 C CNN
+F 2 "azonenberg_pcb:EIA_0402_RES_NOSILK" V 9330 7450 30  0001 C CNN
 F 3 "" H 9400 7450 30  0000 C CNN
 	1    9400 7450
@@
 F 0 "R162" H 10280 7404 50  0000 R CNN
 F 1 "220" H 10280 7496 50  0000 R CNN
-F 2 "" V 10280 7450 30  0001 C CNN
+F 2 "azonenberg_pcb:EIA_0402_RES_NOSILK" V 10280 7450 30  0001 C CNN
 F 3 "" H 10350 7450 30  0000 C CNN
 	1    10350 7450
@@
 F 0 "R164" H 11230 7404 50  0000 R CNN
 F 1 "220" H 11230 7496 50  0000 R CNN
-F 2 "" V 11230 7450 30  0001 C CNN
+F 2 "azonenberg_pcb:EIA_0402_RES_NOSILK" V 11230 7450 30  0001 C CNN
 F 3 "" H 11300 7450 30  0000 C CNN
 	1    11300 7450
@@
 F 0 "R166" H 12180 7404 50  0000 R CNN
 F 1 "220" H 12180 7496 50  0000 R CNN
-F 2 "" V 12180 7450 30  0001 C CNN
+F 2 "azonenberg_pcb:EIA_0402_RES_NOSILK" V 12180 7450 30  0001 C CNN
 F 3 "" H 12250 7450 30  0000 C CNN
 	1    12250 7450
@@
 F 0 "R168" H 13130 7404 50  0000 R CNN
 F 1 "220" H 13130 7496 50  0000 R CNN
-F 2 "" V 13130 7450 30  0001 C CNN
+F 2 "azonenberg_pcb:EIA_0402_RES_NOSILK" V 13130 7450 30  0001 C CNN
 F 3 "" H 13200 7450 30  0000 C CNN
 	1    13200 7450

Commit message: More footprint assignments
Parts:
- R178, R180: footprint (none) -> azonenberg_pcb:EIA_0402_RES_NOSILK
Changed lines of the file:
@@
 F 0 "R178" V 3000 900 50  0000 C CNN
 F 1 "1" V 3100 950 50  0000 C CNN
-F 2 "" V 3030 950 30  0001 C CNN
+F 2 "azonenberg_pcb:EIA_0402_RES_NOSILK" V 3030 950 30  0001 C CNN
 F 3 "" H 3100 950 30  0000 C CNN
 	1    3100 950
@@
 F 0 "R180" V 7500 1550 50  0000 C CNN
 F 1 "1" V 7600 1600 50  0000 C CNN
-F 2 "" V 7530 1600 30  0001 C CNN
+F 2 "azonenberg_pcb:EIA_0402_RES_NOSILK" V 7530 1600 30  0001 C CNN
 F 3 "" H 7600 1600 30  0000 C CNN
 	1    7600 1600

Commit message: Finished component footprints. Ready to begin layout.
Parts:
- U32: footprint (none) -> azonenberg_pcb:DFN_4_0.5MM_1.6x1.2MM
Changed lines of the file:
@@
 Sheet 4 7
 Title "GreenPak Hardware-In-Loop Test Platform"
-Date "2016-05-20"
+Date "2016-05-22"
 Rev "0.1"
 Comp "Andrew Zonenberg"
@@
 F 0 "U32" H 5800 2100 60  0000 C CNN
 F 1 "SIP32408" H 6150 2100 60  0000 C CNN
-F 2 "" H 5750 2150 60  0001 C CNN
+F 2 "azonenberg_pcb:DFN_4_0.5MM_1.6x1.2MM" H 5750 2150 60  0001 C CNN
 F 3 "" H 5750 2150 60  0000 C CNN
 	1    5750 2150

Commit message: Began routing RGMII bus
Parts:
- P1, P2: footprint azonenberg_pcb:CONN_HEADER_2.54MM_2x10_RA_BRORIG -> azonenberg_pcb:CONN_HEADER_2.54MM_2x10_RA_TRORIG
Changed lines of the file:
@@
 Sheet 4 7
 Title "GreenPak Hardware-In-Loop Test Platform"
-Date "2016-05-22"
+Date "2016-05-23"
 Rev "0.1"
 Comp "Andrew Zonenberg"
@@
 F 0 "P1" H 1478 1938 50  0000 L CNN
 F 1 "GPAK_ZIF" H 1478 1846 50  0000 L CNN
-F 2 "azonenberg_pcb:CONN_HEADER_2.54MM_2x10_RA_BRORIG" H 1400 1900 60  0001 C CNN
+F 2 "azonenberg_pcb:CONN_HEADER_2.54MM_2x10_RA_TRORIG" H 1400 1900 60  0001 C CNN
 F 3 "" H 1400 1900 60  0000 C CNN
 	1    1400 1900
@@
 F 0 "P2" H 1478 4388 50  0000 L CNN
 F 1 "2x10 HEADER" H 1478 4296 50  0000 L CNN
-F 2 "azonenberg_pcb:CONN_HEADER_2.54MM_2x10_RA_BRORIG" H 1400 4350 60  0001 C CNN
+F 2 "azonenberg_pcb:CONN_HEADER_2.54MM_2x10_RA_TRORIG" H 1400 4350 60  0001 C CNN
 F 3 "" H 1400 4350 60  0000 C CNN
 	1    1400 4350
