File: boards/gp4-hil/fpga-support.sch (KiCad schematic (older format))
At the start: 77 parts, among them J2 XILINX_JTAG, U2 XC7A100T-1FTG256C, U6 W25Q32FW

Commit message: Began work on footprint creation for layout.
Parts:
- C100, C101, C102, C103, C104, C105, C106, C107, C108, C109, C110, C111, C112, C113, C114, C115, C144, C67, C70, C73, C75, C77, C79, C80, C81, C82, C83, C84, C85, C86: footprint (none) -> azonenberg_pcb:EIA_0402_CAP_NOSILK
- C143, C66, C68, C69, C71, C72, C74, C76, C78, C92, C93, C94, C95, C96, C97, C98, C99: footprint (none) -> azonenberg_pcb:EIA_0603_CAP_NOSILK
- C63, C64: footprint (none) -> azonenberg_pcb:EIA_1210_CAP_NOSILK
- C65, C87, C88, C89, C90, C91: footprint (none) -> azonenberg_pcb:EIA_1206_CAP_NOSILK
- J2: footprint (none) -> azonenberg_pcb:XILINX_JTAG_PTH_MOLEX_0878311420

Commit message: Updated PCB with a lot more component footprints
Parts:
- R119, R120, R121, R122, R123, R124, R125, R126, R127, R128, R129, R130, R131, R132, R133, R134: footprint (none) -> azonenberg_pcb:EIA_0402_RES_NOSILK
- U2: footprint (none) -> azonenberg_pcb:BGA_256_17x17_FULLARRAY_1MM
Changed lines of the file:
@@
 Sheet 6 7
 Title "GreenPak Hardware-In-Loop Test Platform"
-Date "2016-05-19"
+Date "2016-05-20"
 Rev "0.1"
 Comp "Andrew Zonenberg"
@@
 F 0 "U2" H 8050 10750 60  0000 L CNN
 F 1 "XC7A100T-1FTG256C" H 8050 10850 60  0000 L CNN
-F 2 "" H 8050 10950 60  0001 C CNN
+F 2 "azonenberg_pcb:BGA_256_17x17_FULLARRAY_1MM" H 8050 10950 60  0001 C CNN
 F 3 "" H 8050 10950 60  0000 C CNN
 	1    8050 10950
@@
 F 0 "U2" H 11450 10750 60  0000 L CNN
 F 1 "XC7A100T-1FTG256C" H 11450 10850 60  0000 L CNN
-F 2 "" H 11450 10950 60  0001 C CNN
+F 2 "azonenberg_pcb:BGA_256_17x17_FULLARRAY_1MM" H 11450 10950 60  0001 C CNN
 F 3 "" H 11450 10950 60  0000 C CNN
 	2    11450 10950
@@
 F 0 "R121" V 7300 9500 50  0000 C CNN
 F 1 "33" V 7350 9650 50  0000 C CNN
-F 2 "" V 7280 9650 30  0001 C CNN
+F 2 "azonenberg_pcb:EIA_0402_RES_NOSILK" V 7280 9650 30  0001 C CNN
 F 3 "" H 7350 9650 30  0000 C CNN
 	1    7350 9650
@@
 F 0 "R120" V 6700 10550 50  0000 C CNN
 F 1 "1K" V 6750 10350 50  0000 C CNN
-F 2 "" V 6680 10350 30  0001 C CNN
+F 2 "azonenberg_pcb:EIA_0402_RES_NOSILK" V 6680 10350 30  0001 C CNN
 F 3 "" H 6750 10350 30  0000 C CNN
 	1    6750 10350
@@
 F 0 "R119" V 6700 10450 50  0000 C CNN
 F 1 "1K" V 6750 10250 50  0000 C CNN
-F 2 "" V 6680 10250 30  0001 C CNN
+F 2 "azonenberg_pcb:EIA_0402_RES_NOSILK" V 6680 10250 30  0001 C CNN
 F 3 "" H 6750 10250 30  0000 C CNN
 	1    6750 10250
@@
 F 0 "R122" V 17500 8800 50  0000 C CNN
 F 1 "33" V 17550 8600 50  0000 C CNN
-F 2 "" V 17480 8600 30  0001 C CNN
+F 2 "azonenberg_pcb:EIA_0402_RES_NOSILK" V 17480 8600 30  0001 C CNN
 F 3 "" H 17550 8600 30  0000 C CNN
 	1    17550 8600
@@
 F 0 "R123" V 17500 8900 50  0000 C CNN
 F 1 "33" V 17550 8700 50  0000 C CNN
-F 2 "" V 17480 8700 30  0001 C CNN
+F 2 "azonenberg_pcb:EIA_0402_RES_NOSILK" V 17480 8700 30  0001 C CNN
 F 3 "" H 17550 8700 30  0000 C CNN
 	1    17550 8700
@@
 F 0 "R124" V 18150 7600 50  0000 C CNN
 F 1 "33" V 18200 7400 50  0000 C CNN
-F 2 "" V 18130 7400 30  0001 C CNN
+F 2 "azonenberg_pcb:EIA_0402_RES_NOSILK" V 18130 7400 30  0001 C CNN
 F 3 "" H 18200 7400 30  0000 C CNN
 	1    18200 7400
@@
 F 0 "R125" V 18150 7700 50  0000 C CNN
 F 1 "33" V 18200 7500 50  0000 C CNN
-F 2 "" V 18130 7500 30  0001 C CNN
+F 2 "azonenberg_pcb:EIA_0402_RES_NOSILK" V 18130 7500 30  0001 C CNN
 F 3 "" H 18200 7500 30  0000 C CNN
 	1    18200 7500
@@
 F 0 "R126" V 18150 7800 50  0000 C CNN
 F 1 "33" V 18200 7600 50  0000 C CNN
-F 2 "" V 18130 7600 30  0001 C CNN
+F 2 "azonenberg_pcb:EIA_0402_RES_NOSILK" V 18130 7600 30  0001 C CNN
 F 3 "" H 18200 7600 30  0000 C CNN
 	1    18200 7600
@@
 F 0 "R127" V 18150 7900 50  0000 C CNN
 F 1 "33" V 18200 7700 50  0000 C CNN
-F 2 "" V 18130 7700 30  0001 C CNN
+F 2 "azonenberg_pcb:EIA_0402_RES_NOSILK" V 18130 7700 30  0001 C CNN
 F 3 "" H 18200 7700 30  0000 C CNN
 	1    18200 7700
@@
 F 0 "R128" V 18150 8000 50  0000 C CNN
 F 1 "33" V 18200 7800 50  0000 C CNN
-F 2 "" V 18130 7800 30  0001 C CNN
+F 2 "azonenberg_pcb:EIA_0402_RES_NOSILK" V 18130 7800 30  0001 C CNN
 F 3 "" H 18200 7800 30  0000 C CNN
 	1    18200 7800
@@
 F 0 "R133" V 19500 8800 50  0000 C CNN
 F 1 "33" V 19550 8600 50  0000 C CNN
-F 2 "" V 19480 8600 30  0001 C CNN
+F 2 "azonenberg_pcb:EIA_0402_RES_NOSILK" V 19480 8600 30  0001 C CNN
 F 3 "" H 19550 8600 30  0000 C CNN
 	1    19550 8600
@@
 F 0 "R134" V 19500 9000 50  0000 C CNN
 F 1 "33" V 19550 8800 50  0000 C CNN
-F 2 "" V 19480 8800 30  0001 C CNN
+F 2 "azonenberg_pcb:EIA_0402_RES_NOSILK" V 19480 8800 30  0001 C CNN
 F 3 "" H 19550 8800 30  0000 C CNN
 	1    19550 8800
@@
 F 0 "R129" V 18150 8150 50  0000 C CNN
 F 1 "33" V 18200 7950 50  0000 C CNN
-F 2 "" V 18130 7950 30  0001 C CNN
+F 2 "azonenberg_pcb:EIA_0402_RES_NOSILK" V 18130 7950 30  0001 C CNN
 F 3 "" H 18200 7950 30  0000 C CNN
 	1    18200 7950
@@
 F 0 "R132" V 19450 7450 50  0000 C CNN
 F 1 "4.7K" V 19550 7450 50  0000 C CNN
-F 2 "" V 19480 7450 30  0001 C CNN
+F 2 "azonenberg_pcb:EIA_0402_RES_NOSILK" V 19480 7450 30  0001 C CNN
 F 3 "" H 19550 7450 30  0000 C CNN
 	1    19550 7450
@@
 F 0 "R131" V 19250 7350 50  0000 C CNN
 F 1 "4.7K" V 19350 7350 50  0000 C CNN
-F 2 "" V 19280 7350 30  0001 C CNN
+F 2 "azonenberg_pcb:EIA_0402_RES_NOSILK" V 19280 7350 30  0001 C CNN
 F 3 "" H 19350 7350 30  0000 C CNN
 	1    19350 7350
@@
 F 0 "R130" V 19050 7300 50  0000 C CNN
 F 1 "4.7K" V 19150 7250 50  0000 C CNN
-F 2 "" V 19080 7250 30  0001 C CNN
+F 2 "azonenberg_pcb:EIA_0402_RES_NOSILK" V 19080 7250 30  0001 C CNN
 F 3 "" H 19150 7250 30  0000 C CNN
 	1    19150 7250

Commit message: More footprint assignments
Parts:
- R135, R136, R137: footprint (none) -> azonenberg_pcb:EIA_0402_RES_NOSILK
Changed lines of the file:
@@
 F 0 "R135" V 7150 10950 50  0000 C CNN
 F 1 "0" V 7200 10750 50  0000 C CNN
-F 2 "" V 7130 10750 30  0001 C CNN
+F 2 "azonenberg_pcb:EIA_0402_RES_NOSILK" V 7130 10750 30  0001 C CNN
 F 3 "" H 7200 10750 30  0000 C CNN
 	1    7200 10750
@@
 F 0 "R136" V 7150 11050 50  0000 C CNN
 F 1 "0" V 7200 10850 50  0000 C CNN
-F 2 "" V 7130 10850 30  0001 C CNN
+F 2 "azonenberg_pcb:EIA_0402_RES_NOSILK" V 7130 10850 30  0001 C CNN
 F 3 "" H 7200 10850 30  0000 C CNN
 	1    7200 10850
@@
 F 0 "R137" V 7150 11150 50  0000 C CNN
 F 1 "0" V 7200 10950 50  0000 C CNN
-F 2 "" V 7130 10950 30  0001 C CNN
+F 2 "azonenberg_pcb:EIA_0402_RES_NOSILK" V 7130 10950 30  0001 C CNN
 F 3 "" H 7200 10950 30  0000 C CNN
 	1    7200 10950

Commit message: Finished component footprints. Ready to begin layout.
Parts:
- U6: footprint (none) -> azonenberg_pcb:DFN_8_1.27MM_6x5MM
Changed lines of the file:
@@
 Sheet 6 7
 Title "GreenPak Hardware-In-Loop Test Platform"
-Date "2016-05-20"
+Date "2016-05-22"
 Rev "0.1"
 Comp "Andrew Zonenberg"
@@
 F 0 "U6" H 18550 9587 60  0000 C CNN
 F 1 "W25Q32FW" H 18550 9481 60  0000 C CNN
-F 2 "" H 18550 8900 60  0001 C CNN
+F 2 "azonenberg_pcb:DFN_8_1.27MM_6x5MM" H 18550 8900 60  0001 C CNN
 F 3 "" H 18550 8900 60  0000 C CNN
 	1    18550 8900
