File: boards/gp4-hil/analog-io.sch (KiCad schematic (older format))
At the start: 119 parts, among them U10 AD9609, U11 DAC084S085, U12 DAC084S085, U13 DAC084S085, U14 DAC084S085, U19 TS3A4751, U2 XC7A100T-1FTG256C, U25 TS3A4751, U26 TS3A4751, U27 TS3A4751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

Commit message: More ADC layout
Connections:
- net ADC_A_D0: now also U2.E16 (IO_L17P_T2_A26_15); no longer U2.E11 (IO_L14P_T2_SRCC_15)
- net ADC_A_D1: now also U2.F15 (IO_L18P_T2_A24_15); no longer U2.D11 (IO_L14N_T2_SRCC_15)
- net ADC_A_D2: now also U2.G15 (IO_L24N_T3_RS0_15); no longer U2.D14 (IO_L15P_T2_DQS_15)
- net ADC_A_D3: now also U2.G16 (IO_L22N_T3_A16_15); no longer U2.D15 (IO_L15N_T2_DQS_ADV_B_15)
- net ADC_A_D4: now also U2.H16 (IO_L22P_T3_A17_15); no longer U2.F12 (IO_L16P_T2_A28_15)
- net ADC_A_D5: now also U2.H14 (IO_L24P_T3_RS1_15); no longer U2.F13 (IO_L16N_T2_A27_15)
- net ADC_A_D6: now also U2.H13 (IO_L20N_T3_A19_15); no longer U2.E16 (IO_L17P_T2_A26_15)
- net ADC_A_D7: now also U2.G14 (IO_L21P_T3_DQS_15); no longer U2.D16 (IO_L17N_T2_A25_15)
- net ADC_A_D8: now also U2.G12 (IO_L19N_T3_A21_VREF_15); no longer U2.F15 (IO_L18P_T2_A24_15)
- net ADC_A_D9: now also U2.F14 (IO_L21N_T3_DQS_A18_15); no longer U2.E15 (IO_L18N_T2_A23_15)
- net ADC_B_D5: now also U2.E15 (IO_L18N_T2_A23_15); no longer U2.A13 (IO_L7P_T1_AD2P_15)
- net ADC_B_D6: now also U2.D16 (IO_L17N_T2_A25_15); no longer U2.A14 (IO_L7N_T1_AD2N_15)
- net ADC_B_MODE: now also U2.F13 (IO_L16N_T2_A27_15); no longer U2.H14 (IO_L24P_T3_RS1_15)
- net DAC_A_DIN: now also U2.E11 (IO_L14P_T2_SRCC_15); no longer U2.H16 (IO_L22P_T3_A17_15)
- net DAC_B_DIN: now also U2.D11 (IO_L14N_T2_SRCC_15); no longer U2.F14 (IO_L21N_T3_DQS_A18_15)
- net DAC_C_DIN: now also U2.H11 (IO_L19P_T3_A22_15); no longer U2.G14 (IO_L21P_T3_DQS_15)
- net DAC_D_DIN: now also U2.F12 (IO_L16P_T2_A28_15); no longer U2.H13 (IO_L20N_T3_A19_15)
- net DAC_SCLK: now also U2.D14 (IO_L15P_T2_DQS_15); no longer U2.G15 (IO_L24N_T3_RS0_15)
- net DAC_SYNC_N: now also U2.D15 (IO_L15N_T2_DQS_ADV_B_15); no longer U2.G16 (IO_L22N_T3_A16_15)
- net at C152.1, R140.2: now also U2.A14 (IO_L7N_T1_AD2N_15); no longer U2.B16 (IO_L10N_T1_AD11N_15)
- net at C151.1, R140.1: now also U2.A13 (IO_L7P_T1_AD2P_15); no longer U2.C16 (IO_L10P_T1_AD11P_15)
- net at C154.1, R141.2: now also U2.B16 (IO_L10N_T1_AD11N_15); no longer U2.G12 (IO_L19N_T3_A21_VREF_15)
- net at C153.1, R141.1: now also U2.C16 (IO_L10P_T1_AD11P_15); no longer U2.H11 (IO_L19P_T3_A22_15)
Other:
- moved on the sheet: C151, C152, C153, C154, R140, R141
Changed lines of the file:
@@
 Text Label 1150 11800 2    60   ~ 0
 GND
-Text Label 20550 3850 2    60   ~ 0
+Text Label 20550 4450 2    60   ~ 0
 ADC_A_D0
-Text Label 20550 3950 2    60   ~ 0
+Text Label 20550 4650 2    60   ~ 0
 ADC_A_D1
-Text Label 20550 4050 2    60   ~ 0
+Text Label 20550 5950 2    60   ~ 0
 ADC_A_D2
-Text Label 20550 4150 2    60   ~ 0
+Text Label 20550 5550 2    60   ~ 0
 ADC_A_D3
-Text Label 20550 4250 2    60   ~ 0
+Text Label 20550 5450 2    60   ~ 0
 ADC_A_D4
-Text Label 20550 4350 2    60   ~ 0
+Text Label 20550 5850 2    60   ~ 0
 ADC_A_D5
-Text Label 20550 4450 2    60   ~ 0
+Text Label 20550 5150 2    60   ~ 0
 ADC_A_D6
-Text Label 20550 4550 2    60   ~ 0
+Text Label 20550 5250 2    60   ~ 0
 ADC_A_D7
-Text Label 20550 4650 2    60   ~ 0
+Text Label 20550 4950 2    60   ~ 0
 ADC_A_D8
-Text Label 20550 4750 2    60   ~ 0
+Text Label 20550 5350 2    60   ~ 0
 ADC_A_D9
 Text Label 20550 3650 2    60   ~ 0
@@
 Text Label 20550 5050 2    60   ~ 0
 ADC_A_SDIO
-Text Label 18650 4750 2    60   ~ 0
+Text Label 18650 2950 2    60   ~ 0
 ADC_A_CLK_P
-Text Label 18650 5050 2    60   ~ 0
+Text Label 18650 3250 2    60   ~ 0
 ADC_A_CLK_N
 Text Label 20550 1950 2    60   ~ 0
@@
 Text Label 20550 2350 2    60   ~ 0
 ADC_B_D4
-Text Label 20550 2450 2    60   ~ 0
+Text Label 20550 4750 2    60   ~ 0
 ADC_B_D5
-Text Label 20550 2550 2    60   ~ 0
+Text Label 20550 4550 2    60   ~ 0
 ADC_B_D6
 Text Label 20550 2650 2    60   ~ 0
@@
 Text Label 20550 3350 2    60   ~ 0
 ADC_B_SDIO
-Text Label 18650 2950 2    60   ~ 0
+Text Label 18650 2350 2    60   ~ 0
 ADC_B_CLK_P
-Text Label 18650 3250 2    60   ~ 0
+Text Label 18650 2650 2    60   ~ 0
 ADC_B_CLK_N
 NoConn ~ 20650 3750
 NoConn ~ 20650 3550
-Text Label 20550 5550 2    60   ~ 0
+Text Label 20550 4150 2    60   ~ 0
 DAC_SYNC_N
-Text Label 20550 5450 2    60   ~ 0
+Text Label 20550 3850 2    60   ~ 0
 DAC_A_DIN
-Text Label 20550 5350 2    60   ~ 0
+Text Label 20550 3950 2    60   ~ 0
 DAC_B_DIN
-Text Label 20550 5250 2    60   ~ 0
+Text Label 20550 4850 2    60   ~ 0
 DAC_C_DIN
-Text Label 20550 5150 2    60   ~ 0
+Text Label 20550 4250 2    60   ~ 0
 DAC_D_DIN
-Text Label 20550 5950 2    60   ~ 0
+Text Label 20550 4050 2    60   ~ 0
 DAC_SCLK
 $Comp
@@
 L C C151
 U 1 1 574AF1AD
+P 18900 2350
+F 0 "C151" V 18800 2150 50  0000 C CNN
+F 1 "0.1 uF" V 18800 2550 50  0000 C CNN
+F 2 "azonenberg_pcb:EIA_0402_CAP_NOSILK" H 18938 2200 30  0001 C CNN
+F 3 "" H 18900 2350 60  0000 C CNN
+	1    18900 2350
+	0    1    1    0
+$EndComp
+$Comp
+L C C152
+U 1 1 574AF1B3
+P 18900 2650
+F 0 "C152" V 18800 2450 50  0000 C CNN
+F 1 "0.1 uF" V 18800 2850 50  0000 C CNN
+F 2 "azonenberg_pcb:EIA_0402_CAP_NOSILK" H 18938 2500 30  0001 C CNN
+F 3 "" H 18900 2650 60  0000 C CNN
+	1    18900 2650
+	0    1    1    0
+$EndComp
+$Comp
+L R R140
+U 1 1 574B00A3
+P 19300 2500
+F 0 "R140" H 19370 2546 50  0000 L CNN
+F 1 "100" H 19370 2454 50  0000 L CNN
+F 2 "azonenberg_pcb:EIA_0402_RES_NOSILK" V 19230 2500 30  0001 C CNN
+F 3 "" H 19300 2500 30  0000 C CNN
+	1    19300 2500
+	1    0    0    -1
+$EndComp
+$Comp
+L C C153
+U 1 1 574B3A27
 P 18900 2950
-F 0 "C151" V 18800 2750 50  0000 C CNN
+F 0 "C153" V 18800 2750 50  0000 C CNN
 F 1 "0.1 uF" V 18800 3150 50  0000 C CNN
 F 2 "azonenberg_pcb:EIA_0402_CAP_NOSILK" H 18938 2800 30  0001 C CNN
@@
 $EndComp
 $Comp
-L C C152
-U 1 1 574AF1B3
+L C C154
+U 1 1 574B3A2D
 P 18900 3250
-F 0 "C152" V 18800 3050 50  0000 C CNN
+F 0 "C154" V 18800 3050 50  0000 C CNN
 F 1 "0.1 uF" V 18800 3450 50  0000 C CNN
 F 2 "azonenberg_pcb:EIA_0402_CAP_NOSILK" H 18938 3100 30  0001 C CNN
@@
 $EndComp
 $Comp
-L R R140
-U 1 1 574B00A3
+L R R141
+U 1 1 574B3A35
 P 19300 3100
-F 0 "R140" H 19370 3146 50  0000 L CNN
+F 0 "R141" H 19370 3146 50  0000 L CNN
 F 1 "100" H 19370 3054 50  0000 L CNN
 F 2 "azonenberg_pcb:EIA_0402_RES_NOSILK" V 19230 3100 30  0001 C CNN
 F 3 "" H 19300 3100 30  0000 C CNN
 	1    19300 3100
-	1    0    0    -1
-$EndComp
-$Comp
-L C C153
-U 1 1 574B3A27
-P 18900 4750
-F 0 "C153" V 18800 4550 50  0000 C CNN
-F 1 "0.1 uF" V 18800 4950 50  0000 C CNN
-F 2 "azonenberg_pcb:EIA_0402_CAP_NOSILK" H 18938 4600 30  0001 C CNN
-F 3 "" H 18900 4750 60  0000 C CNN
-	1    18900 4750
-	0    1    1    0
-$EndComp
-$Comp
-L C C154
-U 1 1 574B3A2D
-P 18900 5050
-F 0 "C154" V 18800 4850 50  0000 C CNN
-F 1 "0.1 uF" V 18800 5250 50  0000 C CNN
-F 2 "azonenberg_pcb:EIA_0402_CAP_NOSILK" H 18938 4900 30  0001 C CNN
-F 3 "" H 18900 5050 60  0000 C CNN
-	1    18900 5050
-	0    1    1    0
-$EndComp
-$Comp
-L R R141
-U 1 1 574B3A35
-P 19300 4900
-F 0 "R141" H 19370 4946 50  0000 L CNN
-F 1 "100" H 19370 4854 50  0000 L CNN
-F 2 "azonenberg_pcb:EIA_0402_RES_NOSILK" V 19230 4900 30  0001 C CNN
-F 3 "" H 19300 4900 30  0000 C CNN
-	1    19300 4900
 	1    0    0    -1
 $EndComp
@@
 Text Label 1450 14650 2    60   ~ 0
 ADC_B_MODE
-Text Label 20550 5850 2    60   ~ 0
+Text Label 20550 4350 2    60   ~ 0
 ADC_B_MODE
 Text Label 20550 6050 2    60   ~ 0
@@
 	20550 3850 20650 3850
 Wire Wire Line
-	20550 4750 20650 4750
-Wire Wire Line
-	20650 4650 20550 4650
-Wire Wire Line
-	20550 4550 20650 4550
-Wire Wire Line
-	20650 4450 20550 4450
-Wire Wire Line
 	20550 4350 20650 4350
 Wire Wire Line
@@
 	20550 2650 20650 2650
 Wire Wire Line
-	20650 2550 20550 2550
-Wire Wire Line
-	20550 2450 20650 2450
+	20650 4550 20550 4550
+Wire Wire Line
+	20550 4450 20650 4450
 Wire Wire Line
 	20550 2350 20650 2350
@@
 Connection ~ 5650 9300
 Wire Wire Line
+	19750 2450 20650 2450
+Wire Wire Line
+	19750 2550 20650 2550
+Wire Wire Line
+	19050 2650 19750 2650
+Wire Wire Line
+	19750 2650 19750 2550
+Wire Wire Line
+	19050 2350 19750 2350
+Wire Wire Line
+	19750 2350 19750 2450
+Wire Wire Line
 	19750 3050 20650 3050
 Wire Wire Line
 	19750 3150 20650 3150
 Wire Wire Line
+	19750 3250 19750 3150
+Wire Wire Line
+	19750 2950 19750 3050
+Wire Wire Line
+	18650 2350 18750 2350
+Connection ~ 19300 2350
+Connection ~ 19300 2650
+Wire Wire Line
+	18750 2650 18650 2650
+Wire Wire Line
 	19050 3250 19750 3250
 Wire Wire Line
-	19750 3250 19750 3150
-Wire Wire Line
 	19050 2950 19750 2950
-Wire Wire Line
-	19750 2950 19750 3050
-Wire Wire Line
-	19750 4850 20650 4850
-Wire Wire Line
-	19750 4950 20650 4950
-Wire Wire Line
-	19750 5050 19750 4950
-Wire Wire Line
-	19750 4750 19750 4850
 Wire Wire Line
 	18650 2950 18750 2950
@@
 Wire Wire Line
 	18750 3250 18650 3250
-Wire Wire Line
-	19050 5050 19750 5050
-Wire Wire Line
-	19050 4750 19750 4750
-Wire Wire Line
-	18650 4750 18750 4750
-Connection ~ 19300 4750
-Connection ~ 19300 5050
-Wire Wire Line
-	18750 5050 18650 5050
 Wire Wire Line
 	800  9600 1150 9600
@@
 Text HLabel 1450 13050 0    60   Input ~ 0
 2V5
+Wire Wire Line
+	20550 4950 20650 4950
+Wire Wire Line
+	20550 4650 20650 4650
+Wire Wire Line
+	20650 4850 20550 4850
+Wire Wire Line
+	20550 4750 20650 4750
 $EndSCHEMATC

Commit message: Continued work on GreenPak test board
Connections:
- net ADC_A_D8: now also U2.H12 (IO_L20P_T3_A20_15); no longer U2.G12 (IO_L19N_T3_A21_VREF_15)
- net ADC_A_MODE: now also U2.C12 (IO_L11N_T1_SRCC_15); no longer U2.G11 (IO_25_15)
- net ADC_A_SDIO: now also U2.C13 (IO_L12N_T1_MRCC_15); no longer U2.H12 (IO_L20P_T3_A20_15)
- net ADC_B_D0: now also U2.E15 (IO_L18N_T2_A23_15); no longer U2.B11 (IO_L4N_T0_15)
- net ADC_B_D1: now also U2.D16 (IO_L17N_T2_A25_15); no longer U2.B12 (IO_L5P_T0_AD9P_15)
- net ADC_B_D2: now also U2.B15 (IO_L9P_T1_DQS_AD3P_15); no longer U2.A12 (IO_L5N_T0_AD9N_15)
- net ADC_B_D3: now also U2.C16 (IO_L10P_T1_AD11P_15); no longer U2.D8 (IO_L6P_T0_15)
- net ADC_B_D4: now also U2.B16 (IO_L10N_T1_AD11N_15); no longer U2.D9 (IO_L6N_T0_VREF_15)
- net ADC_B_D5: now also U2.A15 (IO_L9N_T1_DQS_AD3N_15); no longer U2.E15 (IO_L18N_T2_A23_15)
- net ADC_B_D6: now also U2.B14 (IO_L8N_T1_AD10N_15); no longer U2.D16 (IO_L17N_T2_A25_15)
- net ADC_B_D7: now also U2.G12 (IO_L19N_T3_A21_VREF_15); no longer U2.C14 (IO_L8P_T1_AD10P_15)
- net ADC_B_D8: now also U2.C14 (IO_L8P_T1_AD10P_15); no longer U2.B14 (IO_L8N_T1_AD10N_15)
- net ADC_B_D9: now also U2.F13 (IO_L16N_T2_A27_15); no longer U2.B15 (IO_L9P_T1_DQS_AD3P_15)
- net ADC_B_MODE: now also U2.A12 (IO_L5N_T0_AD9N_15); no longer U2.F13 (IO_L16N_T2_A27_15)
- net ADC_B_SDIO: now also U2.A14 (IO_L7N_T1_AD2N_15); no longer U2.C12 (IO_L11N_T1_SRCC_15)
- net ADC_CS_N: now also U2.B12 (IO_L5P_T0_AD9P_15); no longer U2.A15 (IO_L9N_T1_DQS_AD3N_15)
- net ADC_GPIO20: now also U8.32 (S8B); no longer U8.30 (S6B)
- net ADC_SCLK: now also U2.A13 (IO_L7P_T1_AD2P_15); no longer U2.C11 (IO_L11P_T1_SRCC_15)
- net ADC_VDD2: now also U8.30 (S6B); no longer U8.32 (S8B)
- net DAC_C_DIN: now also U2.D9 (IO_L6N_T0_VREF_15); no longer U2.H11 (IO_L19P_T3_A22_15)
- net DAC_SCLK: now also U2.D8 (IO_L6P_T0_15); no longer U2.D14 (IO_L15P_T2_DQS_15)
- net DAC_SYNC_N: now also U2.C11 (IO_L11P_T1_SRCC_15); no longer U2.D15 (IO_L15N_T2_DQS_ADV_B_15)
- net MUX_A3: now also U2.B11 (IO_L4N_T0_15); no longer U2.A8 (IO_L2P_T0_AD8P_15)
- net MUX_CS_A_N: now also U2.G11 (IO_25_15); no longer U2.A9 (IO_L2N_T0_AD8N_15)
- net ADC_B_CLKX_P: now reaches C151.1, R140.1
- net ADC_B_CLKX_P: now also U2.A8 (IO_L2P_T0_AD8P_15); no longer U2.A13 (IO_L7P_T1_AD2P_15)
- net ADC_B_CLKX_N: now reaches C152.1, R140.2
- net ADC_B_CLKX_N: now also U2.A9 (IO_L2N_T0_AD8N_15); no longer U2.A14 (IO_L7N_T1_AD2N_15)
- net ADC_A_CLKX_N: now reaches C154.1, R141.2
- net ADC_A_CLKX_N: now also U2.D15 (IO_L15N_T2_DQS_ADV_B_15); no longer U2.B16 (IO_L10N_T1_AD11N_15)
- net ADC_A_CLKX_P: now reaches C153.1, R141.1
- net ADC_A_CLKX_P: now also U2.D14 (IO_L15P_T2_DQS_15); no longer U2.C16 (IO_L10P_T1_AD11P_15)
Other:
- moved on the sheet: C151, C152, C153, C154, R140, R141
Changed lines of the file:
@@
 Sheet 5 7
 Title "GreenPak Hardware-In-Loop Test Platform"
-Date "2016-06-04"
+Date "2016-06-05"
 Rev "0.1"
 Comp "Andrew Zonenberg"
@@
 Text Label 20550 1350 2    60   ~ 0
 MUX_A2
-Text Label 20550 1450 2    60   ~ 0
+Text Label 20550 1950 2    60   ~ 0
 MUX_A3
-Text Label 20550 1550 2    60   ~ 0
+Text Label 20550 6050 2    60   ~ 0
 MUX_CS_A_N
 Text Label 20550 1650 2    60   ~ 0
@@
 Text Label 20550 5250 2    60   ~ 0
 ADC_A_D7
-Text Label 20550 4950 2    60   ~ 0
+Text Label 20550 5050 2    60   ~ 0
 ADC_A_D8
 Text Label 20550 5350 2    60   ~ 0
@@
 Text Label 20550 3650 2    60   ~ 0
 ADC_A_DCLK
-Text Label 20550 2950 2    60   ~ 0
+Text Label 20550 2050 2    60   ~ 0
 ADC_CS_N
-Text Label 20550 3250 2    60   ~ 0
+Text Label 20550 2450 2    60   ~ 0
 ADC_SCLK
-Text Label 20550 5050 2    60   ~ 0
+Text Label 20550 3550 2    60   ~ 0
 ADC_A_SDIO
-Text Label 18650 2950 2    60   ~ 0
+Text Label 18650 3950 2    60   ~ 0
 ADC_A_CLK_P
-Text Label 18650 3250 2    60   ~ 0
+Text Label 18650 4250 2    60   ~ 0
 ADC_A_CLK_N
-Text Label 20550 1950 2    60   ~ 0
+Text Label 20550 4750 2    60   ~ 0
 ADC_B_D0
-Text Label 20550 2050 2    60   ~ 0
+Text Label 20550 4550 2    60   ~ 0
 ADC_B_D1
-Text Label 20550 2150 2    60   ~ 0
+Text Label 20550 2850 2    60   ~ 0
 ADC_B_D2
-Text Label 20550 2250 2    60   ~ 0
+Text Label 20550 3050 2    60   ~ 0
 ADC_B_D3
-Text Label 20550 2350 2    60   ~ 0
+Text Label 20550 3150 2    60   ~ 0
 ADC_B_D4
-Text Label 20550 4750 2    60   ~ 0
+Text Label 20550 2950 2    60   ~ 0
 ADC_B_D5
-Text Label 20550 4550 2    60   ~ 0
+Text Label 20550 2750 2    60   ~ 0
 ADC_B_D6
-Text Label 20550 2650 2    60   ~ 0
+Text Label 20550 4950 2    60   ~ 0
 ADC_B_D7
-Text Label 20550 2750 2    60   ~ 0
+Text Label 20550 2650 2    60   ~ 0
 ADC_B_D8
-Text Label 20550 2850 2    60   ~ 0
+Text Label 20550 4350 2    60   ~ 0
 ADC_B_D9
 Text Label 20550 3450 2    60   ~ 0
 ADC_B_DCLK
-Text Label 20550 3350 2    60   ~ 0
+Text Label 20550 2550 2    60   ~ 0
 ADC_B_SDIO
-Text Label 18650 2350 2    60   ~ 0
+Text Label 18650 1350 2    60   ~ 0
 ADC_B_CLK_P
-Text Label 18650 2650 2    60   ~ 0
+Text Label 18650 1650 2    60   ~ 0
 ADC_B_CLK_N
-NoConn ~ 20650 3750
-NoConn ~ 20650 3550
-Text Label 20550 4150 2    60   ~ 0
+Text Label 20550 3250 2    60   ~ 0
 DAC_SYNC_N
 Text Label 20550 3850 2    60   ~ 0
@@
 Text Label 20550 3950 2    60   ~ 0
 DAC_B_DIN
-Text Label 20550 4850 2    60   ~ 0
+Text Label 20550 2350 2    60   ~ 0
 DAC_C_DIN
 Text Label 20550 4250 2    60   ~ 0
 DAC_D_DIN
-Text Label 20550 4050 2    60   ~ 0
+Text Label 20550 2250 2    60   ~ 0
 DAC_SCLK
 $Comp
@@
 L C C151
 U 1 1 574AF1AD
-P 18900 2350
-F 0 "C151" V 18800 2150 50  0000 C CNN
-F 1 "0.1 uF" V 18800 2550 50  0000 C CNN
-F 2 "azonenberg_pcb:EIA_0402_CAP_NOSILK" H 18938 2200 30  0001 C CNN
-F 3 "" H 18900 2350 60  0000 C CNN
-	1    18900 2350
+P 18900 1350
+F 0 "C151" V 18800 1150 50  0000 C CNN
+F 1 "0.1 uF" V 18800 1550 50  0000 C CNN
+F 2 "azonenberg_pcb:EIA_0402_CAP_NOSILK" H 18938 1200 30  0001 C CNN
+F 3 "" H 18900 1350 60  0000 C CNN
+	1    18900 1350
 	0    1    1    0
 $EndComp
@@
 L C C152
 U 1 1 574AF1B3
-P 18900 2650
-F 0 "C152" V 18800 2450 50  0000 C CNN
-F 1 "0.1 uF" V 18800 2850 50  0000 C CNN
-F 2 "azonenberg_pcb:EIA_0402_CAP_NOSILK" H 18938 2500 30  0001 C CNN
-F 3 "" H 18900 2650 60  0000 C CNN
-	1    18900 2650
+P 18900 1650
+F 0 "C152" V 18800 1450 50  0000 C CNN
+F 1 "0.1 uF" V 18800 1850 50  0000 C CNN
+F 2 "azonenberg_pcb:EIA_0402_CAP_NOSILK" H 18938 1500 30  0001 C CNN
+F 3 "" H 18900 1650 60  0000 C CNN
+	1    18900 1650
 	0    1    1    0
 $EndComp
@@
 L R R140
 U 1 1 574B00A3
-P 19300 2500
-F 0 "R140" H 19370 2546 50  0000 L CNN
-F 1 "100" H 19370 2454 50  0000 L CNN
-F 2 "azonenberg_pcb:EIA_0402_RES_NOSILK" V 19230 2500 30  0001 C CNN
-F 3 "" H 19300 2500 30  0000 C CNN
-	1    19300 2500
+P 19300 1500
+F 0 "R140" H 19370 1546 50  0000 L CNN
+F 1 "100" H 19370 1454 50  0000 L CNN
+F 2 "azonenberg_pcb:EIA_0402_RES_NOSILK" V 19230 1500 30  0001 C CNN
+F 3 "" H 19300 1500 30  0000 C CNN
+	1    19300 1500
 	1    0    0    -1
 $EndComp
@@
 L C C153
 U 1 1 574B3A27
-P 18900 2950
-F 0 "C153" V 18800 2750 50  0000 C CNN
-F 1 "0.1 uF" V 18800 3150 50  0000 C CNN
-F 2 "azonenberg_pcb:EIA_0402_CAP_NOSILK" H 18938 2800 30  0001 C CNN
-F 3 "" H 18900 2950 60  0000 C CNN
-	1    18900 2950
+P 18900 3950
+F 0 "C153" V 18800 3750 50  0000 C CNN
+F 1 "0.1 uF" V 18800 4150 50  0000 C CNN
+F 2 "azonenberg_pcb:EIA_0402_CAP_NOSILK" H 18938 3800 30  0001 C CNN
+F 3 "" H 18900 3950 60  0000 C CNN
+	1    18900 3950
 	0    1    1    0
 $EndComp
@@
 L C C154
 U 1 1 574B3A2D
-P 18900 3250
-F 0 "C154" V 18800 3050 50  0000 C CNN
-F 1 "0.1 uF" V 18800 3450 50  0000 C CNN
-F 2 "azonenberg_pcb:EIA_0402_CAP_NOSILK" H 18938 3100 30  0001 C CNN
-F 3 "" H 18900 3250 60  0000 C CNN
-	1    18900 3250
+P 18900 4250
+F 0 "C154" V 18800 4050 50  0000 C CNN
+F 1 "0.1 uF" V 18800 4450 50  0000 C CNN
+F 2 "azonenberg_pcb:EIA_0402_CAP_NOSILK" H 18938 4100 30  0001 C CNN
+F 3 "" H 18900 4250 60  0000 C CNN
+	1    18900 4250
 	0    1    1    0
 $EndComp
@@
 L R R141
 U 1 1 574B3A35
-P 19300 3100
-F 0 "R141" H 19370 3146 50  0000 L CNN
-F 1 "100" H 19370 3054 50  0000 L CNN
-F 2 "azonenberg_pcb:EIA_0402_RES_NOSILK" V 19230 3100 30  0001 C CNN
-F 3 "" H 19300 3100 30  0000 C CNN
-	1    19300 3100
+P 19300 4100
+F 0 "R141" H 19370 4146 50  0000 L CNN
+F 1 "100" H 19370 4054 50  0000 L CNN
+F 2 "azonenberg_pcb:EIA_0402_RES_NOSILK" V 19230 4100 30  0001 C CNN
+F 3 "" H 19300 4100 30  0000 C CNN
+	1    19300 4100
 	1    0    0    -1
 $EndComp
@@
 Text Label 1450 14650 2    60   ~ 0
 ADC_B_MODE
-Text Label 20550 4350 2    60   ~ 0
+Text Label 20550 2150 2    60   ~ 0
 ADC_B_MODE
-Text Label 20550 6050 2    60   ~ 0
+Text Label 20550 3350 2    60   ~ 0
 ADC_A_MODE
 Text Label 6250 4150 2    60   ~ 0
@@
 	1    0    0    -1
 $EndComp
-Text Notes 18650 3450 0    60   ~ 0
+Text Notes 18850 1850 0    60   ~ 0
 LVDS_25
 $Comp
@@
 	20550 1250 20650 1250
 Wire Wire Line
-	20550 1450 20650 1450
+	20550 2450 20650 2450
 Wire Wire Line
 	20650 1350 20550 1350
 Wire Wire Line
-	20550 1550 20650 1550
+	20550 2550 20650 2550
 Wire Wire Line
 	20550 1850 20650 1850
@@
 	20550 3850 20650 3850
 Wire Wire Line
-	20550 4350 20650 4350
+	20550 4950 20650 4950
 Wire Wire Line
 	20550 4250 20650 4250
 Wire Wire Line
-	20650 4150 20550 4150
+	20650 3150 20550 3150
 Wire Wire Line
-	20550 4050 20650 4050
+	20550 3050 20650 3050
 Wire Wire Line
 	20650 3950 20550 3950
 Wire Wire Line
-	20550 5050 20650 5050
+	20550 3550 20650 3550
 Wire Wire Line
 	20550 5150 20650 5150
@@
 Connection ~ 5650 9300
 Wire Wire Line
-	19750 2450 20650 2450
+	19750 1450 20650 1450
 Wire Wire Line
-	19750 2550 20650 2550
+	19750 1550 20650 1550
 Wire Wire Line
-	19050 2650 19750 2650
+	19050 1650 19750 1650
 Wire Wire Line
-	19750 2650 19750 2550
+	19750 1650 19750 1550
 Wire Wire Line
-	19050 2350 19750 2350
+	19050 1350 19750 1350
 Wire Wire Line
-	19750 2350 19750 2450
+	19750 1350 19750 1450
 Wire Wire Line
-	19750 3050 20650 3050
+	19750 4050 20650 4050
 Wire Wire Line
-	19750 3150 20650 3150
+	19750 4150 20650 4150
 Wire Wire Line
-	19750 3250 19750 3150
+	19750 4250 19750 4150
 Wire Wire Line
-	19750 2950 19750 3050
+	19750 3950 19750 4050
 Wire Wire Line
-	18650 2350 18750 2350
-Connection ~ 19300 2350
-Connection ~ 19300 2650
+	18650 1350 18750 1350
+Connection ~ 19300 1350
+Connection ~ 19300 1650
 Wire Wire Line
-	18750 2650 18650 2650
+	18750 1650 18650 1650
 Wire Wire Line
-	19050 3250 19750 3250
+	19050 4250 19750 4250
 Wire Wire Line
-	19050 2950 19750 2950
+	19050 3950 19750 3950
 Wire Wire Line
-	18650 2950 18750 2950
-Connection ~ 19300 2950
-Connection ~ 19300 3250
+	18650 3950 18750 3950
+Connection ~ 19300 3950
+Connection ~ 19300 4250
 Wire Wire Line
-	18750 3250 18650 3250
+	18750 4250 18650 4250
 Wire Wire Line
 	800  9600 1150 9600
@@
 Text Label 3150 5650 0    60   ~ 0
 ADC_GPIO2
-Text Label 3150 5750 0    60   ~ 0
+Text Label 3150 5950 0    60   ~ 0
 ADC_GPIO20
 Text Label 3150 5850 0    60   ~ 0
 ADC_VDD1
-Text Label 3150 5950 0    60   ~ 0
+Text Label 3150 5750 0    60   ~ 0
 ADC_VDD2
 Wire Wire Line
@@
 2V5
 Wire Wire Line
-	20550 4950 20650 4950
+	20550 5050 20650 5050
 Wire Wire Line
 	20550 4650 20650 4650
 Wire Wire Line
-	20650 4850 20550 4850
+	20650 4350 20550 4350
 Wire Wire Line
 	20550 4750 20650 4750
+Text Label 20550 1450 2    60   ~ 0
+ADC_B_CLKX_P
+Text Label 20550 1550 2    60   ~ 0
+ADC_B_CLKX_N
+Text Label 20550 4050 2    60   ~ 0
+ADC_A_CLKX_P
+Text Label 20550 4150 2    60   ~ 0
+ADC_A_CLKX_N
+NoConn ~ 20650 4850
+NoConn ~ 20650 3750
 $EndSCHEMATC
