File: boards/gp4-stqfn20-thermal/gp4-stqfn20-thermal.kicad_pcb (KiCad board)
At the start: 4 copper layers, 37 x 28 mm, 15 parts, among them J1 GREENPAK_ZIF_HDR, P1 CONN_01X04, U1 SI7050, U2 INA226, U3 SLG46620V

Commit message: Updated design after review
Parts:
- moved G*** 1.00 mm to (91.5, 64.5)
Other:
- board text added: "3V3"
- board text added: "GND"
- board text added: "SCL"
- board text added: "SDA"
Changed lines of the file:
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@@
     (area 72.03375 46.948214 112.85375 78.80375)
     (thickness 1.6)
-    (drawings 7)
+    (drawings 11)
     (tracks 2527)
     (zones 0)
@@
     (visible_elements FFFDFF7F)
     (pcbplotparams
-      (layerselection 0x00030_ffffffff)
+      (layerselection 0x010fc_ffffffff)
       (usegerberextensions false)
       (excludeedgelayer true)
@@
       (outputformat 1)
       (mirror false)
-      (drillshape 1)
+      (drillshape 0)
       (scaleselection 1)
-      (outputdirectory ""))
+      (outputdirectory output/))
   )
   (net 0 "")
@@
   )
   (module azonenberg_pcb:LONGTHING-1200DPI (layer B.Cu)
-    (at 91.5 65.5 180)
+    (at 91.5 64.5 180)
     (fp_text reference G*** (at 3 2 180) (layer B.SilkS) hide
       (effects (font (thickness 0.3)) (justify mirror))
@@
   (module azonenberg_pcb:EIA_0603_CAP_NOSILK (layer B.Cu)
     (at 89 72)
-    (fp_text reference C1 (at 0 -1.5) (layer B.SilkS)
+    (fp_text reference C1 (at 0 1.5) (layer B.SilkS)
       (effects (font (size 0.75 0.75) (thickness 0.125)) (justify mirror))
     )
@@
     )
   )
+  (gr_text 3V3 (at 88.25 71.5 270) (layer B.SilkS)
+    (effects (font (size 1 1) (thickness 0.125)) (justify left mirror))
+  )
+  (gr_text SDA (at 90.75 71.5 270) (layer B.SilkS)
+    (effects (font (size 1 1) (thickness 0.125)) (justify left mirror))
+  )
+  (gr_text SCL (at 93.25 71.5 270) (layer B.SilkS)
+    (effects (font (size 1 1) (thickness 0.125)) (justify left mirror))
+  )
+  (gr_text GND (at 95.75 71.5 270) (layer B.SilkS)
+    (effects (font (size 1 1) (thickness 0.125)) (justify left mirror))
+  )
   (gr_text "DIE #" (at 98.6 73.6) (layer F.SilkS)

Commit message: Updated gp4-stqfn-thermal with correct pinout for 20-pin header (PCB rev 0.2)
Parts:
- J1: footprint azonenberg_pcb:CONN_HEADER_2.54MM_2x10_RA_FEMALE -> azonenberg_pcb:CONN_HEADER_2.54MM_2x10_RA_TRORIG
Routing:
- net /GND: track 90.8 -> 85.0 mm
- net /VDD_IN: track 13.2 -> 9.70 mm
- net /DUT_P13: track 36.7 -> 40.0 mm
- net /DUT_P10: track 37.0 -> 40.1 mm
- net /DUT_P20: track 37.0 -> 40.1 mm
- net /DUT_P15: track 37.0 -> 40.1 mm
- net /DUT_P9: track 37.0 -> 40.1 mm
- net /DUT_P6: track 37.0 -> 40.1 mm
- net /DUT_P2: track 37.8 -> 40.9 mm
- net /DUT_P4: track 37.0 -> 40.0 mm
- net /DUT_P12: track 37.0 -> 40.0 mm
- net /DUT_P17: track 37.1 -> 40.1 mm
- net /DUT_P8: track 37.0 -> 40.0 mm
- net /DUT_P19: track 37.0 -> 40.0 mm
- net /DUT_P14: track 37.0 -> 40.0 mm
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Other:
- board text added: "GreenPAK STQFN-20 v0.2 Thermal Characterization A. Zonenberg / 2017-07-11"
- board text removed: "GreenPAK STQFN-20 Thermal Characterization A. Zonenberg / 2017-06-22"
