File: boards/gp4-stqfn20-thermal/gp4-stqfn20-thermal.sch (KiCad schematic (older format))
At the start: 11 parts, among them J1 GREENPAK_ZIF_HDR, P1 CONN_01X04, U1 SI7050, U2 INA226, U3 SLG46620V

Commit message: Updated design after review
Parts:
- R1: footprint (none) -> azonenberg_pcb:EIA_0805_CAP_NOSILK
- U1: footprint (none) -> azonenberg_pcb:DFN_6_1MM_3x3MM
- U3: footprint (none) -> azonenberg_pcb:QFN_20_0.4MM_3x2MM_SILEGO_STQFN
Changed lines of the file:
@@
 F 0 "U1" H 2100 5047 60  0000 C CNN
 F 1 "SI7050" H 2100 4941 60  0000 C CNN
-F 2 "" H 2000 4550 60  0001 C CNN
+F 2 "azonenberg_pcb:DFN_6_1MM_3x3MM" H 2000 4550 60  0001 C CNN
 F 3 "" H 2000 4550 60  0001 C CNN
 	1    1850 4650
@@
 F 0 "U3" H 5900 2900 60  0000 L CNN
 F 1 "SLG46620V" H 5900 2800 60  0000 L CNN
-F 2 "" H 5900 2950 60  0001 C CNN
+F 2 "azonenberg_pcb:QFN_20_0.4MM_3x2MM_SILEGO_STQFN" H 5900 2950 60  0001 C CNN
 F 3 "" H 5900 2950 60  0001 C CNN
 	1    5900 2950
@@
 F 0 "R1" V 2950 900 50  0000 C CNN
 F 1 "1" V 3050 900 50  0000 C CNN
-F 2 "" V 2980 900 50  0000 C CNN
+F 2 "azonenberg_pcb:EIA_0805_CAP_NOSILK" V 2980 900 50  0001 C CNN
 F 3 "" H 3050 900 50  0000 C CNN
 	1    3050 900

Commit message: Updated schematic for v0.2 thermal board
Parts:
- J1: footprint azonenberg_pcb:CONN_HEADER_2.54MM_2x10_RA_FEMALE -> azonenberg_pcb:CONN_HEADER_2.54MM_2x10_RA_TRORIG
Changed lines of the file:
@@
 F 0 "J1" H 2450 2800 60  0000 R CNN
 F 1 "GREENPAK_ZIF_HDR" H 2450 2900 60  0000 R CNN
-F 2 "azonenberg_pcb:CONN_HEADER_2.54MM_2x10_RA_FEMALE" H 1950 2900 60  0001 C CNN
+F 2 "azonenberg_pcb:CONN_HEADER_2.54MM_2x10_RA_TRORIG" H 1950 2900 60  0001 C CNN
 F 3 "" H 1950 2900 60  0001 C CNN
 	1    1950 2950
